Commit message: add moveit config

File: black_maine_description/urdf/black_maine_robot.urdf.xacro (robot description, xacro)
@@ -21,6 +21,6 @@
   </link>
   <joint name="body_joint" type="fixed">
-    <origin xyz="0 0 0.075" rpy="0 0 0" />
-    <parent link="base_link"/>
+    <origin xyz="0 0 0.0884" rpy="0 0 0" />
+    <parent link="base_footprint"/>
     <child link="body_link"/>
   </joint>

Commit message: add panel

File: black_maine_description/urdf/black_maine_robot.urdf.xacro (robot description, xacro)
@@ -37,5 +37,5 @@
   </link>
   <joint name="arm_base_joint" type="fixed">
-    <origin xyz="0.121 0 0.057" rpy="0 0 0" />
+    <origin xyz="0.121 0 0.081" rpy="0 0 0" />
     <parent link="body_link"/>
     <child link="arm_base_link"/>
